File: KiCAD/PETRAMROM.kicad_pcb (KiCad board)
At the start: 2 copper layers, 87 x 62.2 mm, 21 parts, among them SW1 DIP, SW2 ROMSEL, U0 SOCKET, U1 MOS6502, U2 74LS245, U3 62256, U4 SST39SF040, U5 GAL16V8

Commit message: Add files via upload
Parts:
- U5: value GAL16V8 -> ATF16V8
Changed lines of the file:
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@@
       (effects (font (size 1 1) (thickness 0.15)))
     )
-    (fp_text value GAL16V8 (at 3.81 17.145 270) (layer F.Fab)
+    (fp_text value ATF16V8 (at 3.81 17.145 270) (layer F.Fab)
       (effects (font (size 1 1) (thickness 0.15)))
     )
