File: KiCAD/PETRAMROM.sch (KiCad schematic (older format))
At the start: 21 parts, among them SW1 DIP, SW2 ROMSEL, U0 SOCKET, U1 MOS6502, U2 74LS245, U3 62256, U4 SST39SF040, U5 GAL16V8

Commit message: Add files via upload
Parts:
- U5: value GAL16V8 -> ATF16V8
Changed lines of the file:
@@
 P 2750 4950
 F 0 "U5" H 2750 5828 50  0000 C CNN
-F 1 "GAL16V8" H 2750 5737 50  0000 C CNN
+F 1 "ATF16V8" H 2750 5737 50  0000 C CNN
 F 2 "Package_DIP:DIP-20_W7.62mm_LongPads" H 2750 4950 50  0001 C CNN
 F 3 "" H 2750 4950 50  0001 C CNN
